Commit message: Add files via upload

File: src/chronos_balance/urdf/chronos.urdf (robot description, URDF)
Before this commit: robot chronos, 40 links, 39 joints
Joints:
- joint Lower_Leg_v2_v1_Revolute_91: limit lower=-0.523599 upper=0.523599 effort=1000000 velocity=1000000 -> lower=-1.04 upper=1.04 effort=1000000 velocity=1000000
- joint ankle_joint_ring1_a_Revolute_119: limit lower=-0.349066 upper=0.349066 effort=1000000 velocity=1000000 -> lower=-0.7 upper=0.7 effort=1000000 velocity=1000000
- joint ankle_joint_ring1_b_Revolute_115: limit lower=-0.349066 upper=0.349066 effort=1000000 velocity=1000000 -> lower=-0.7 upper=0.7 effort=1000000 velocity=1000000
- joint leg_knee_motor_a_Revolute_74: limit lower=-1.570796 upper=0.0 effort=1000000 velocity=1000000 -> lower=-2.1 upper=0.0 effort=1000000 velocity=1000000
- joint leg_knee_motor_v1_Revolute_82: limit lower=0.0 upper=1.570796 effort=1000000 velocity=1000000 -> lower=0.0 upper=2.1 effort=1000000 velocity=1000000
- joint lower_leg_right_v1_Revolute_69: limit lower=-0.523599 upper=0.523599 effort=1000000 velocity=1000000 -> lower=-1.04 upper=1.04 effort=1000000 velocity=1000000
- joint motor_upper_a_Rigid_35: limit lower=-0.4 upper=0.4 effort=20 velocity=5 -> lower=-0.7 upper=0.7 effort=20 velocity=5
- joint motor_upper_b_Rigid_131: limit lower=-0.4 upper=0.4 effort=20 velocity=5 -> lower=-0.7 upper=0.7 effort=20 velocity=5
- joint motor_upper_leg_below_a_v1_Revolute_123: limit lower=-0.785398 upper=0.785398 effort=1000000 velocity=1000000 -> lower=-1.5 upper=1.5 effort=1000000 velocity=1000000
- joint motor_upper_leg_below_v1_Revolute_31: limit lower=-0.785398 upper=0.785398 effort=1000000 velocity=1000000 -> lower=-1.5 upper=1.5 effort=1000000 velocity=1000000
